File: doc/kicad/rover.kicad_sch (KiCad schematic)
At the start: 4 parts, among them J1 I2C, J2 UART, J3 UART, U1 STM32F411_BlackPill

Commit message: Update schematic
Parts:
- added U2: ESP32_C3, RF_Module:WEMOS_D1_mini_light, symbol DRX:ESP32_C3_TENSTAR
Connections:
- net GND: now also U1.19 (G); no longer U1.20 (5V)
- net at J2.1 (RX), U1.32 (A12): now also U2.16 (P7)
- net at J2.2 (TX), U1.33 (A11): now also U2.15 (P6)
- net +5V: no longer names the net of U1.23 (5V)
Other:
- moved on the sheet: U1

Commit message: Update schematic
Parts:
- added M1, M2, M3, M4: DC_Motor_Enc_5pin, symbol DRX:DC_Motor_Enc_5pin
- added U3: LSM303DLHC, Package_LGA:LGA-14_3x5mm_P0.8mm_LayoutBorder1x6y, symbol Sensor_Motion:LSM303DLHC
Connections:
- net GND: now also U2.7 (G), M2.4 (GND), M4.4 (GND), U3.10 (GND), U3.11 (GND), U3.7 (GND)
- net 5V: now reaches U1.23 (5V)
- net 5V: now also U2.6 (5V)
- net at J1.1 (SDA), U1.26 (B7): now also U3.3 (SDA)
- net at J1.2 (SCL), U1.27 (B6): now also U3.2 (SCL)
- new net 3.3: M2.3 (VCC), M4.3 (VCC)
- new net 3.3V: U3.14 (VDD)
- new net L_ENC: M4.5 (OUT)
- new net L_MOTOR_A: M1.1 (M+), M2.1 (M+)
- new net L_MOTOR_B: M1.2 (M-), M2.2 (M-)
- new net R_ENC: M2.5 (OUT)
- new net R_MOTOR_A: M3.1 (M+), M4.1 (M+)
- new net R_MOTOR_B: M3.2 (M-), M4.2 (M-)
- no-connect marks 0 -> 6
Other:
- note added: "Left"
- note added: "Main board: Vehicle controller, radio, IMU"
- note added: "Motor connections"
- note added: "Right"
- title: Rover main board -> Rover prototype modules
- moved on the sheet: U1

Commit message: Improve motor control
Parts:
- added U4: L298N_Breakout_E, symbol DRX:L298N_Breakout_Expanded
- added U5: AMS1117-3.3, Package_TO_SOT_SMD:SOT-223-3_TabPin2, symbol Regulator_Linear:AMS1117-3.3
- added U6: ~, symbol DRX:Rover_PowerBus1
Connections:
- net 3.3 is gone; now on net 3.3V: M2.3 (VCC), M4.3 (VCC)
- net 3.3V: now also U5.2 (VO)
- net 5V: now also U4.13 (5V), U5.3 (VI), U6.1 (VCC), U6.3 (VOUT1)
- net GND: now also U4.12 (GND), U5.1 (GND), U6.2 (GND), U6.6 (GND)
- net L_MOTOR_A: now also U4.8 (M1B)
- net L_MOTOR_B: now also U4.7 (M1A)
- net R_MOTOR_A: now also U4.10 (M2B)
- net R_MOTOR_B: now also U4.9 (M2A)
- net MOTOR_B_EN: now reaches U1.3 (C14)
- net MOTOR_B_EN: now also U4.6 (ENB)
- net MOTOR_A_EN: now reaches U1.4 (C15)
- net MOTOR_A_EN: now also U4.1 (ENA)
- net PWM_1: now reaches U1.6 (A0)
- net PWM_1: now also U4.2 (IN1)
- net PWM_2: now reaches U1.7 (A1)
- net PWM_2: now also U4.3 (IN2)
- net PWM_3: now reaches U1.8 (A2)
- net PWM_3: now also U4.4 (IN3)
- net PWM_4: now reaches U1.9 (A3)
- net PWM_4: now also U4.5 (IN4)
- new net VBATT: U4.11 (VMS)
Other:
- moved on the sheet: U1, U2, U3
